Commit message: test of ignition fisics

File: src/caramelo_description/URDF/lidar_sensor.xacro (robot description, xacro)
@@ -16,7 +16,12 @@
         <origin xyz="0 0 0" rpy="0 0 0"/>
       </collision>
-      <xacro:inertial_cylinder mass="0.1" length="0.016" radius="0.030">
-        <origin xyz="0 0 0" />
-      </xacro:inertial_cylinder>
+      <inertial>
+        <origin xyz="0 0 0" rpy="0 0 0"/>
+        <mass value="0.1"/>
+        <inertia
+          ixx="1e-5" ixy="0.0" ixz="0.0"
+          iyy="1e-5" iyz="0.0"
+          izz="1e-5"/>
+      </inertial>
     </link>
     <joint name="laser_joint" type="fixed">
@@ -26,5 +31,4 @@
     </joint>
     <gazebo reference="laser_frame">
-      <material>Gazebo/Red</material>
       <sensor name="rplidar" type="ray">
         <pose>0 0 0 0 0 0</pose>
@@ -44,7 +48,6 @@
           </range>
         </ray>
-        <plugin name="laser_controller" filename="libgazebo_ros2_laser_sensor.so">
-          <ros_topic>/scan</ros_topic>
-          <output_type>sensor_msgs/LaserScan</output_type>
+        <plugin name="gazebo_ros_ray_sensor" filename="libignition-gazebo-ros-ray-system.so">
+          <topic>/scan</topic>
           <frame_name>laser_frame</frame_name>
         </plugin>

File: src/caramelo_description/URDF/robot_mecanum_wheel.xacro (robot description, xacro)
@@ -1,4 +1,4 @@
 <?xml version="1.0"?>
-<robot xmlns:xacro="http://www.ros.org/wiki/xacro">
+<robot xmlns:xacro="http://www.ros.org/wiki/xacro" xmlns:ignition="http://gazebosim.org/schema">
   <xacro:property name="wheel_radius" value="0.05"/>
   <xacro:property name="wheel_width" value="0.075"/>
@@ -42,4 +42,5 @@
               <mu>1.0</mu>
               <mu2>1.0</mu2>
+              <fdir1>${x_reflect} ${y_reflect} 0</fdir1>
           </ode>
         </friction>
