Commit message: Controller mecanum v1

File: src/caramelo_description/URDF/robot.urdf.xacro (robot description, xacro)
@@ -1,6 +1,7 @@
 <?xml version="1.0"?>
 <robot name="caramelo" xmlns:xacro="http://ros.org/wiki/xacro">
-  <!-- Modelos para simular o robo-->
+  <xacro:arg name="is_ignition" default="true"/>
   <xacro:include filename="robot_core.xacro" />
-  <!-- Controle ros2_control para rodas Mecanum -->
+  <xacro:include filename="robot_gazebo.xacro" />
+  <xacro:include filename="robot_ros2_control.xacro" />
 </robot>

File: src/caramelo_description/URDF/robot_core.xacro (robot description, xacro)
@@ -45,6 +45,5 @@
         </xacro:inertial_box>
     </link>
-    <!--? JOINT ?-->
-    <joint name="base_footprint_to_base_link" type="fixed">
+    <joint name="footprint_to_base_link" type="fixed">
         <parent link="base_footprint" />
         <child link="base_link" />
@@ -54,6 +53,5 @@
         <material>Gazebo\Black</material>
     </gazebo>
-    <!--! FRONT LEFT WHEELS !-->
-    <!--? LINK ?-->
+    <!--! FRONT LEFT WHEEL -->
     <link name="front_left_wheel">
         <visual>
@@ -68,4 +66,5 @@
                 <cylinder radius="0.05" length="0.075" />
             </geometry>
+            <origin rpy="-1.57 0 0" xyz="0 0 0" />
         </collision>
         <xacro:inertial_cylinder mass="0.1" length="0.075" radius="0.05">
@@ -73,6 +72,5 @@
         </xacro:inertial_cylinder>
     </link>
-    <!--? JOINT ?-->
-    <joint name="base_fl_wheel_joint" type="continuous">
+    <joint name="fl_wheel_joint" type="continuous">
         <parent link="base_link" />
         <child link="front_left_wheel" />
@@ -83,6 +81,5 @@
         <material>Gazebo\Blue</material>
     </gazebo>
-    <!--! FRONT RIGHT WHEELS !-->
-    <!--? LINK ?-->
+    <!--! FRONT RIGHT WHEEL -->
     <link name="front_right_wheel">
         <visual>
@@ -97,4 +94,5 @@
                 <cylinder radius="0.05" length="0.075" />
             </geometry>
+            <origin rpy="-1.57 0 0" xyz="0 0 0" />
         </collision>
         <xacro:inertial_cylinder mass="0.1" length="0.075" radius="0.05">
@@ -102,6 +100,5 @@
         </xacro:inertial_cylinder>
     </link>
-    <!--? JOINT ?-->
-    <joint name="base_fr_wheel_joint" type="continuous">
+    <joint name="fr_wheel_joint" type="continuous">
         <parent link="base_link" />
         <child link="front_right_wheel" />
@@ -112,6 +109,5 @@
         <material>Gazebo\Blue</material>
     </gazebo>
-    <!--! REAR LEFT WHEELS !-->
-    <!--? LINK ?-->
+    <!--! REAR LEFT WHEEL -->
     <link name="rear_left_wheel">
         <visual>
@@ -126,4 +122,5 @@
                 <cylinder radius="0.05" length="0.075" />
             </geometry>
+            <origin rpy="-1.57 0 0" xyz="0 0 0" />
         </collision>
         <xacro:inertial_cylinder mass="0.1" length="0.075" radius="0.05">
@@ -131,6 +128,5 @@
         </xacro:inertial_cylinder>
     </link>
-    <!--? JOINT ?-->
-    <joint name="base_rl_wheel_joint" type="continuous">
+    <joint name="rl_wheel_joint" type="continuous">
         <parent link="base_link" />
         <child link="rear_left_wheel" />
@@ -141,6 +137,5 @@
         <material>Gazebo\Blue</material>
     </gazebo>
-    <!--! REAR RIGHT WHEELS !-->
-    <!--? LINK ?-->
+    <!--! REAR RIGHT WHEEL -->
     <link name="rear_right_wheel">
         <visual>
@@ -155,4 +150,5 @@
                 <cylinder radius="0.05" length="0.075" />
             </geometry>
+            <origin rpy="-1.57 0 0" xyz="0 0 0" />
         </collision>
         <xacro:inertial_cylinder mass="0.1" length="0.075" radius="0.05">
@@ -160,6 +156,5 @@
         </xacro:inertial_cylinder>
     </link>
-    <!--? JOINT ?-->
-    <joint name="base_rr_wheel_joint" type="continuous">
+    <joint name="rr_wheel_joint" type="continuous">
         <parent link="base_link" />
         <child link="rear_right_wheel" />

Commit message: Update configuration and launch files

File: src/caramelo_description/URDF/robot.urdf.xacro (robot description, xacro)
@@ -5,3 +5,4 @@
   <xacro:include filename="robot_gazebo.xacro" />
   <xacro:include filename="robot_ros2_control.xacro" />
+  <xacro:include filename="inertial_macros.xacro" />
 </robot>

File: src/caramelo_description/URDF/robot_gazebo.xacro (robot description, xacro)
@@ -1,53 +1,55 @@
 <?xml version="1.0"?>
-<robot xmlns:xacro="http://ros.org/wiki/xacro">
-    <gazebo reference="front_left_wheel_link">
-        <mu1>1.0</mu1>
-        <mu2>1.0</mu2>
-        <kp>1e6</kp>
-        <kd>1.0</kd>
-        <minDepth>0.001</minDepth>
-        <maxVel>0.5</maxVel>
-        <fdir1>0.7071 -0.7071 0</fdir1>
-    </gazebo>
-    <gazebo reference="front_right_wheel_link">
-        <mu1>1.0</mu1>
-        <mu2>1.0</mu2>
-        <kp>1e6</kp>
-        <kd>1.0</kd>
-        <minDepth>0.001</minDepth>
-        <maxVel>0.5</maxVel>
-        <fdir1>0.7071 0.7071 0</fdir1>
-    </gazebo>
-    <gazebo reference="rear_left_wheel_link">
-        <mu1>1.0</mu1>
-        <mu2>1.0</mu2>
-        <kp>1e6</kp>
-        <kd>1.0</kd>
-        <minDepth>0.001</minDepth>
-        <maxVel>0.5</maxVel>
-        <fdir1>0.7071 0.7071 0</fdir1>
-    </gazebo>
-    <gazebo reference="rear_right_wheel_link">
-        <mu1>1.0</mu1>
-        <mu2>1.0</mu2>
-        <kp>1e6</kp>
-        <kd>1.0</kd>
-        <minDepth>0.001</minDepth>
-        <maxVel>0.5</maxVel>
-        <fdir1>0.7071 -0.7071 0</fdir1>
-    </gazebo>
-    <gazebo>
-        <!-- ros2 humble -->
-        <xacro:if value="$(arg is_ignition)">
-            <plugin filename="ign_ros2_control-system" name="ign_ros2_control::IgnitionROS2ControlPlugin">
-                <parameters>$(find caramelo_controller)/config/robot_controllers.yaml</parameters>
-            </plugin>
-        </xacro:if>
-        <!-- ros2 newer versions -->
-        <xacro:unless value="$(arg is_ignition)">
-            <plugin filename="gz_ros2_control-system" name="gz_ros2_control::GazeboSimROS2ControlPlugin">
-                <parameters>$(find caramelo_controller)/config/robot_controllers.yaml</parameters>
-            </plugin>
-        </xacro:unless>
-    </gazebo>
+<robot name="caramelo" xmlns:xacro="http://ros.org/wiki/xacro">
+  <!-- Fricção nas rodas Mecanum -->
+  <gazebo reference="front_left_wheel">
+    <mu1>1000000.0</mu1>
+    <mu2>1000000.0</mu2>
+    <kp>1000000.0</kp>
+    <kd>10.0</kd>
+    <minDepth>0.001</minDepth>
+    <maxVel>0.1</maxVel>
+    <fdir1>1 0 0</fdir1>
+  </gazebo>
+  <gazebo reference="front_right_wheel">
+    <mu1>1000000.0</mu1>
+    <mu2>1000000.0</mu2>
+    <kp>1000000.0</kp>
+    <kd>10.0</kd>
+    <minDepth>0.001</minDepth>
+    <maxVel>0.1</maxVel>
+    <fdir1>1 0 0</fdir1>
+  </gazebo>
+  <gazebo reference="rear_left_wheel">
+    <mu1>1000000.0</mu1>
+    <mu2>1000000.0</mu2>
+    <kp>1000000.0</kp>
+    <kd>10.0</kd>
+    <minDepth>0.001</minDepth>
+    <maxVel>0.1</maxVel>
+    <fdir1>1 0 0</fdir1>
+  </gazebo>
+  <gazebo reference="rear_right_wheel">
+    <mu1>1000000.0</mu1>
+    <mu2>1000000.0</mu2>
+    <kp>1000000.0</kp>
+    <kd>10.0</kd>
+    <minDepth>0.001</minDepth>
+    <maxVel>0.1</maxVel>
+    <fdir1>1 0 0</fdir1>
+  </gazebo>
+  <!-- Plugin ROS 2 Control Gazebo -->
+  <gazebo>
+    <!-- ROS 2 Humble -->
+    <xacro:if value="$(arg is_ignition)">
+      <plugin filename="ign_ros2_control-system" name="ign_ros2_control::IgnitionROS2ControlPlugin">
+        <parameters>$(find caramelo_controller)/config/robot_controllers.yaml</parameters>
+      </plugin>
+    </xacro:if>
+    <!-- ROS 2 Iron ou superior -->
+    <xacro:unless value="$(arg is_ignition)">
+      <plugin filename="gz_ros2_control-system" name="gz_ros2_control::GazeboSimROS2ControlPlugin">
+        <parameters>$(find caramelo_controller)/config/robot_controllers.yaml</parameters>
+      </plugin>
+    </xacro:unless>
+  </gazebo>
 </robot>

File: src/caramelo_description/URDF/robot_ros2_control.xacro (robot description, xacro)
@@ -1,31 +1,35 @@
 <?xml version="1.0"?>
-<robot xmlns:xacro="http://ros.org/wiki/xacro">
-  <ros2_control name="RobotSystem" type="system">
-    <xacro:if value="$(arg is_ignition)">
-      <hardware>
-        <plugin>ign_ros2_control/IgnitionSystem</plugin>
-      </hardware>
-    </xacro:if>
-    <xacro:unless value="$(arg is_ignition)">
-      <hardware>
-        <plugin>gz_ros2_control/GazeboSimSystem</plugin>
-      </hardware>
-    </xacro:unless>
-    <joint name="fl_wheel_joint">
-      <command_interface name="velocity"/>
-      <state_interface name="velocity"/>
-    </joint>
-    <joint name="fr_wheel_joint">
-      <command_interface name="velocity"/>
-      <state_interface name="velocity"/>
-    </joint>
-    <joint name="rl_wheel_joint">
-      <command_interface name="velocity"/>
-      <state_interface name="velocity"/>
-    </joint>
-    <joint name="rr_wheel_joint">
-      <command_interface name="velocity"/>
-      <state_interface name="velocity"/>
-    </joint>
-  </ros2_control>
+<robot xmlns:xacro="http://www.ros.org/wiki/xacro" name="caramelo">
+    <ros2_control name="RobotSystem" type="system">
+        <!-- Plugin do ROS 2 Control compatível com Gazebo -->
+        <!-- ROS 2 Humble usa ign_ros2_control -->
+        <xacro:if value="$(arg is_ignition)">
+            <hardware>
+                <plugin>ign_ros2_control/IgnitionSystem</plugin>
+            </hardware>
+        </xacro:if>
+        <!-- ROS 2 Iron ou superior usa gz_ros2_control -->
+        <xacro:unless value="$(arg is_ignition)">
+            <hardware>
+                <plugin>gz_ros2_control/GazeboSimSystem</plugin>
+            </hardware>
+        </xacro:unless>
+        <!-- Declaração dos joints com interface de velocidade -->
+        <joint name="fl_wheel_joint">
+            <command_interface name="velocity" />
+            <state_interface name="velocity" />
+        </joint>
+        <joint name="fr_wheel_joint">
+            <command_interface name="velocity" />
+            <state_interface name="velocity" />
+        </joint>
+        <joint name="rl_wheel_joint">
+            <command_interface name="velocity" />
+            <state_interface name="velocity" />
+        </joint>
+        <joint name="rr_wheel_joint">
+            <command_interface name="velocity" />
+            <state_interface name="velocity" />
+        </joint>
+    </ros2_control>
 </robot>

Commit message: new robot description

File: src/caramelo_description/URDF/robot.urdf.xacro (robot description, xacro)
@@ -1,8 +1,36 @@
 <?xml version="1.0"?>
 <robot name="caramelo" xmlns:xacro="http://ros.org/wiki/xacro">
+  <!-- Argumento para Gazebo Ignition ou Gazebo Classic -->
   <xacro:arg name="is_ignition" default="true"/>
-  <xacro:include filename="robot_core.xacro" />
-  <xacro:include filename="robot_gazebo.xacro" />
+  <!-- Inclusões -->
+  <xacro:include filename="robot_base.xacro" />
+  <xacro:include filename="robot_mecanum_wheel.xacro" />
+  <xacro:include filename="lidar_sensor.xacro" />
   <xacro:include filename="robot_ros2_control.xacro" />
-  <xacro:include filename="inertial_macros.xacro" />
+  <!-- base_footprint -->
+  <link name="base_footprint"/>
+  <!-- Base -->
+  <xacro:robot_base parent="base_footprint"/>
+  <!-- Rodas mecanum -->
+  <xacro:mecanum_wheel prefix="" side="fl" x_reflect="1" y_reflect="1"/>
+  <xacro:mecanum_wheel prefix="" side="fr" x_reflect="1" y_reflect="-1"/>
+  <xacro:mecanum_wheel prefix="" side="rl" x_reflect="-1" y_reflect="1"/>
+  <xacro:mecanum_wheel prefix="" side="rr" x_reflect="-1" y_reflect="-1"/>
+  <!-- LiDAR -->
+  <xacro:lidar_sensor parent="base_link" xyz="0.273 0.012 0.07" rpy="0 0 0"/>
+  <!-- Plugin ROS 2 Control Gazebo -->
+  <gazebo>
+    <!-- ROS 2 Humble -->
+    <xacro:if value="$(arg is_ignition)">
+      <plugin filename="ign_ros2_control-system" name="ign_ros2_control::IgnitionROS2ControlPlugin">
+        <parameters>$(find caramelo_controller)/config/robot_controllers.yaml</parameters>
+      </plugin>
+    </xacro:if>
+    <!-- ROS 2 Iron ou superior -->
+    <xacro:unless value="$(arg is_ignition)">
+      <plugin filename="gz_ros2_control-system" name="gz_ros2_control::GazeboSimROS2ControlPlugin">
+        <parameters>$(find caramelo_controller)/config/robot_controllers.yaml</parameters>
+      </plugin>
+    </xacro:unless>
+  </gazebo>
 </robot>

Commit message: remove caramelo_simulation

File: src/caramelo_description/URDF/robot.urdf.xacro (robot description, xacro)
@@ -1,4 +1,9 @@
 <?xml version="1.0"?>
 <robot name="caramelo" xmlns:xacro="http://ros.org/wiki/xacro">
+  <!-- Propriedades -->
+  <xacro:property name="M_PI" value="3.1415926535897931" />
+  <!-- Argumentos -->
+  <xacro:arg name="robot_name" default="caramelo"/>
+  <xacro:arg name="prefix" default=""/>
   <!-- Argumento para Gazebo Ignition ou Gazebo Classic -->
   <xacro:arg name="is_ignition" default="true"/>
@@ -13,24 +18,33 @@
   <xacro:robot_base parent="base_footprint"/>
   <!-- Rodas mecanum -->
-  <xacro:mecanum_wheel prefix="" side="fl" x_reflect="1" y_reflect="1"/>
-  <xacro:mecanum_wheel prefix="" side="fr" x_reflect="1" y_reflect="-1"/>
-  <xacro:mecanum_wheel prefix="" side="rl" x_reflect="-1" y_reflect="1"/>
-  <xacro:mecanum_wheel prefix="" side="rr" x_reflect="-1" y_reflect="-1"/>
+  <xacro:mecanum_wheel
+    prefix="$(arg prefix)"
+    side="front_left"
+    x_reflect="1"
+    y_reflect="1"/>
+  <xacro:mecanum_wheel
+    prefix="$(arg prefix)"
+    side="front_right"
+    x_reflect="1"
+    y_reflect="-1"/>
+  <xacro:mecanum_wheel
+    prefix="$(arg prefix)"
+    side="back_left"
+    x_reflect="-1"
+    y_reflect="1"/>
+  <xacro:mecanum_wheel
+    prefix="$(arg prefix)"
+    side="back_right"
+    x_reflect="-1"
+    y_reflect="-1"/>
   <!-- LiDAR -->
   <xacro:lidar_sensor parent="base_link" xyz="0.273 0.012 0.07" rpy="0 0 0"/>
   <!-- Plugin ROS 2 Control Gazebo -->
   <gazebo>
-    <!-- ROS 2 Humble -->
-    <xacro:if value="$(arg is_ignition)">
-      <plugin filename="ign_ros2_control-system" name="ign_ros2_control::IgnitionROS2ControlPlugin">
-        <parameters>$(find caramelo_controller)/config/robot_controllers.yaml</parameters>
-      </plugin>
-    </xacro:if>
-    <!-- ROS 2 Iron ou superior -->
-    <xacro:unless value="$(arg is_ignition)">
-      <plugin filename="gz_ros2_control-system" name="gz_ros2_control::GazeboSimROS2ControlPlugin">
-        <parameters>$(find caramelo_controller)/config/robot_controllers.yaml</parameters>
-      </plugin>
-    </xacro:unless>
+    <!-- ROS 2 Jazzy com Gazebo Harmonic -->
+    <plugin filename="gz_ros2_control-system" name="gz_ros2_control::GazeboSimROS2ControlPlugin">
+      <parameters>$(find caramelo_controller)/config/robot_controllers.yaml</parameters>
+      <controller_manager_node_name>controller_manager</controller_manager_node_name>
+    </plugin>
   </gazebo>
 </robot>

File: src/caramelo_description/URDF/robot_mecanum_wheel.xacro (robot description, xacro)
@@ -1,11 +1,14 @@
 <?xml version="1.0"?>
-<robot xmlns:xacro="http://www.ros.org/wiki/xacro" >
-  <xacro:property name="wheel_radius" value="0.05"/>
-  <xacro:property name="wheel_width" value="0.075"/>
-  <xacro:property name="wheel_mass" value="1.0"/>
+<robot xmlns:xacro="http://www.ros.org/wiki/xacro">
+  <xacro:property name="wheel_radius" value="0.05" />
+  <xacro:property name="wheel_width" value="0.075" />
+  <xacro:property name="wheel_mass" value="1.5" />
+  <xacro:property name="wheel_separation" value="0.305" />
+  <xacro:property name="wheel_xoff" value="0.228" />
+  <xacro:property name="wheel_yoff" value="0.0" />
   <xacro:macro name="mecanum_wheel" params="prefix side x_reflect y_reflect">
     <link name="${prefix}${side}_wheel_link">
       <visual>
-        <origin xyz="0 0 0" rpy="${-pi/2} 0 0"/>
+        <origin xyz="0 0 0" rpy="${pi/2} 0 0"/>
         <geometry>
           <cylinder radius="${wheel_radius}" length="${wheel_width}"/>
@@ -16,5 +19,5 @@
       </visual>
       <collision>
-        <origin xyz="0 0 0" rpy="${-pi/2} 0 0"/>
+        <origin xyz="0 0 0" rpy="${pi/2} 0 0"/>
         <geometry>
           <cylinder radius="${wheel_radius}" length="${wheel_width}"/>
@@ -37,20 +40,21 @@
     </joint>
     <gazebo reference="${prefix}${side}_wheel_link">
-      <mu1>1000000000000000.0</mu1>
-      <mu2>1000000000000000.0</mu2>
-      <kp>1000000000000.0</kp>
-      <kd>10.0</kd>
-      <minDepth>0.001</minDepth>
-      <maxVel>0.1</maxVel>
-      <fdir1>${x_reflect} ${y_reflect} 0</fdir1>
+      <surface>
+        <friction>
+          <ode>
+              <mu>1.0</mu>
+              <mu2>1.0</mu2>
+          </ode>
+        </friction>
+      </surface>
       <visual>
-        <material>
-          <ambient>1.0 0.4 0.0 1.0</ambient>
-          <diffuse>1.0 0.4 0.0 1.0</diffuse>
-          <specular>0.2 0.2 0.2 1.0</specular>
-          <emissive>0.0 0.0 0.0 0.0</emissive>
-        </material>
+          <material>
+              <ambient>0.2 0.2 0.2 1.0</ambient>
+              <diffuse>0.2 0.2 0.2 1.0</diffuse>
+              <specular>0.2 0.2 0.2 1.0</specular>
+              <emissive>0.0 0.0 0.0 0.0</emissive>
+          </material>
       </visual>
-    </gazebo>
+  </gazebo>
   </xacro:macro>
 </robot>

File: src/caramelo_description/URDF/robot_ros2_control.xacro (robot description, xacro)
@@ -2,33 +2,40 @@
 <robot xmlns:xacro="http://www.ros.org/wiki/xacro" name="caramelo">
     <ros2_control name="RobotSystem" type="system">
-        <!-- Plugin do ROS 2 Control compatível com Gazebo -->
-        <!-- ROS 2 Humble usa ign_ros2_control -->
-        <xacro:if value="$(arg is_ignition)">
-            <hardware>
-                <plugin>ign_ros2_control/IgnitionSystem</plugin>
-            </hardware>
-        </xacro:if>
-        <!-- ROS 2 Iron ou superior usa gz_ros2_control -->
-        <xacro:unless value="$(arg is_ignition)">
-            <hardware>
-                <plugin>gz_ros2_control/GazeboSimSystem</plugin>
-            </hardware>
-        </xacro:unless>
+        <!-- Plugin do ROS 2 Control compatível com Gazebo Harmonic -->
+        <hardware>
+            <plugin>gz_ros2_control/GazeboSimSystem</plugin>
+        </hardware>
         <!-- Declaração dos joints com interface de velocidade -->
-        <joint name="fl_wheel_joint">
-            <command_interface name="velocity" />
-            <state_interface name="velocity" />
+        <joint name="front_left_wheel_joint">
+            <command_interface name="velocity">
+                <param name="min">-50.0</param>
+                <param name="max">50.0</param>
+            </command_interface>
+            <state_interface name="position"/>
+            <state_interface name="velocity"/>
         </joint>
-        <joint name="fr_wheel_joint">
-            <command_interface name="velocity" />
-            <state_interface name="velocity" />
+        <joint name="front_right_wheel_joint">
+            <command_interface name="velocity">
+                <param name="min">-50.0</param>
+                <param name="max">50.0</param>
+            </command_interface>
+            <state_interface name="position"/>
+            <state_interface name="velocity"/>
         </joint>
-        <joint name="rl_wheel_joint">
-            <command_interface name="velocity" />
-            <state_interface name="velocity" />
+        <joint name="back_left_wheel_joint">
+            <command_interface name="velocity">
+                <param name="min">-50.0</param>
+                <param name="max">50.0</param>
+            </command_interface>
+            <state_interface name="position"/>
+            <state_interface name="velocity"/>
         </joint>
-        <joint name="rr_wheel_joint">
-            <command_interface name="velocity" />
-            <state_interface name="velocity" />
+        <joint name="back_right_wheel_joint">
+            <command_interface name="velocity">
+                <param name="min">-50.0</param>
+                <param name="max">50.0</param>
+            </command_interface>
+            <state_interface name="position"/>
+            <state_interface name="velocity"/>
         </joint>
     </ros2_control>
