Commit message: youbot_description pkg

File: src/caramelo_description/URDF/robot.urdf.xacro (robot description, xacro)
@@ -9,8 +9,8 @@
   <xacro:arg name="is_ignition" default="true"/>
   <!-- Inclusões -->
-  <xacro:include filename="robot_base.xacro" />
-  <xacro:include filename="robot_mecanum_wheel.xacro" />
-  <xacro:include filename="lidar_sensor.xacro" />
-  <xacro:include filename="robot_ros2_control.xacro" />
+  <xacro:include filename="$(find caramelo_description)/URDF/robot_base.xacro" />
+  <xacro:include filename="$(find caramelo_description)/URDF/robot_mecanum_wheel.xacro" />
+  <xacro:include filename="$(find caramelo_description)/URDF/lidar_sensor.xacro" />
+  <xacro:include filename="$(find caramelo_description)/URDF/robot_ros2_control.xacro" />
   <!-- base_footprint -->
   <link name="base_footprint"/>
@@ -38,13 +38,5 @@
     x_reflect="-1"
     y_reflect="-1"/>
-  <!-- LiDAR -->
-  <xacro:lidar_sensor parent="base_link" xyz="0.273 0.012 0.07" rpy="0 0 0"/>
-  <!-- Plugin ROS 2 Control Gazebo -->
-  <gazebo>
-    <!-- ROS 2 Jazzy com Gazebo Harmonic -->
-    <plugin filename="gz_ros2_control-system" name="gz_ros2_control::GazeboSimROS2ControlPlugin">
-      <parameters>$(find caramelo_controller)/config/robot_controllers.yaml</parameters>
-      <controller_manager_node_name>controller_manager</controller_manager_node_name>
-    </plugin>
-  </gazebo>
+  <!-- LiDAR (ajustado para as dimensões do YouBot) -->
+  <xacro:lidar_sensor parent="base_link" xyz="0.290 0.0 0.120" rpy="0 0 0"/>
 </robot>

File: src/caramelo_description/URDF/robot_base.xacro (robot description, xacro)
@@ -2,9 +2,9 @@
 <robot xmlns:xacro="http://www.ros.org/wiki/xacro">
   <xacro:macro name="robot_base" params="parent">
-    <!-- Propriedades -->
-    <xacro:property name="mass" value="25.0"/>
-    <xacro:property name="width" value="0.545"/>
-    <xacro:property name="depth" value="0.225"/>
-    <xacro:property name="height" value="0.140"/>
+    <!-- Propriedades da base do robô Caramelo -->
+    <xacro:property name="mass" value="22.0"/>
+    <xacro:property name="width" value="0.580"/>   <!-- Comprimento -->
+    <xacro:property name="depth" value="0.380"/>   <!-- Largura -->
+    <xacro:property name="height" value="0.105"/>  <!-- Altura -->
     <xacro:property name="wheel_radius" value="0.05"/>
     <!-- Link da base (base_link agora toca o chão) -->
@@ -35,9 +35,9 @@
       </inertial>
     </link>
-    <!-- Joint com o footprint (ajustado para elevar o base_link ao nível do solo) -->
+    <!-- Joint com o footprint (ajustado para as dimensões do Caramelo) -->
     <joint name="base_joint" type="fixed">
       <parent link="${parent}"/>
       <child link="base_link"/>
-      <origin xyz="0 0 ${wheel_radius - 0.02}" rpy="0 0 0"/>
+      <origin xyz="0 0 ${wheel_radius - 0.01}" rpy="0 0 0"/>
     </joint>
     <!-- Aparência no Gazebo -->

File: src/caramelo_description/URDF/robot_mecanum_wheel.xacro (robot description, xacro)
@@ -1,21 +1,23 @@
 <?xml version="1.0"?>
 <robot xmlns:xacro="http://www.ros.org/wiki/xacro">
+  <!-- Especificações das rodas mecanum do robô Caramelo -->
   <xacro:property name="wheel_radius" value="0.05" />
-  <xacro:property name="wheel_width" value="0.075" />
-  <xacro:property name="wheel_mass" value="1.5" />
-  <xacro:property name="wheel_separation" value="0.305" />
-  <xacro:property name="wheel_xoff" value="0.228" />
-  <xacro:property name="wheel_yoff" value="0.0" />
+  <xacro:property name="wheel_width" value="0.061" />
+  <xacro:property name="wheel_mass" value="3.0" />
+  <xacro:property name="wheel_separation" value="0.370" />
+  <xacro:property name="wheel_base" value="0.470" />
   <xacro:macro name="mecanum_wheel" params="prefix side x_reflect y_reflect">
     <link name="${prefix}${side}_wheel_link">
+      <!-- Geometria visual: roda como cilindro -->
       <visual>
-        <origin xyz="0 0 0" rpy="${pi/2} 0 0"/>
+        <origin xyz="0 0 0" rpy="0 0 0"/>
         <geometry>
           <cylinder radius="${wheel_radius}" length="${wheel_width}"/>
         </geometry>
-        <material name="orange">
-          <color rgba="1.0 0.4 0.0 1.0"/>
+        <material name="wheel_material">
+          <color rgba="0.8 0.8 0.0 1.0"/>
         </material>
       </visual>
+      <!-- Geometria de colisão: cilindro simples para otimização de performance -->
       <collision>
         <origin xyz="0 0 0" rpy="${pi/2} 0 0"/>
@@ -24,4 +26,5 @@
         </geometry>
       </collision>
+      <!-- Propriedades inerciais baseadas no cilindro -->
       <inertial>
         <origin xyz="0 0 0" rpy="0 0 0"/>
@@ -33,28 +36,18 @@
       </inertial>
     </link>
+    <!-- Joint da roda: rotação contínua em torno do eixo Y -->
     <joint name="${prefix}${side}_wheel_joint" type="continuous">
       <axis xyz="0 1 0"/>
       <parent link="${prefix}base_link"/>
       <child link="${prefix}${side}_wheel_link"/>
-      <origin xyz="${x_reflect*0.237} ${y_reflect*0.150} 0.02" rpy="0 0 0"/>
+      <origin xyz="${x_reflect*(wheel_base/2)} ${y_reflect*(wheel_separation/2)} 0" rpy="0 0 0"/>
     </joint>
+    <!-- Configurações específicas do Gazebo para as rodas mecanum -->
     <gazebo reference="${prefix}${side}_wheel_link">
-      <surface>
-        <friction>
-          <ode>
-              <mu>1.0</mu>
-              <mu2>1.0</mu2>
-          </ode>
-        </friction>
-      </surface>
-      <visual>
-          <material>
-              <ambient>0.2 0.2 0.2 1.0</ambient>
-              <diffuse>0.2 0.2 0.2 1.0</diffuse>
-              <specular>0.2 0.2 0.2 1.0</specular>
-              <emissive>0.0 0.0 0.0 0.0</emissive>
-          </material>
-      </visual>
-  </gazebo>
+      <material>Gazebo/DarkGrey</material>
+      <!-- Propriedades de fricção básicas - configuração simplificada -->
+      <mu1>1.0</mu1>
+      <mu2>1.0</mu2>
+    </gazebo>
   </xacro:macro>
 </robot>

File: src/caramelo_description/URDF/robot_ros2_control.xacro (robot description, xacro)
@@ -1,4 +1,5 @@
 <?xml version="1.0"?>
 <robot xmlns:xacro="http://www.ros.org/wiki/xacro" name="caramelo">
+    <!-- ros2_control configuration for Caramelo mecanum drive robot -->
     <ros2_control name="RobotSystem" type="system">
         <!-- Plugin do ROS 2 Control compatível com Gazebo Harmonic -->
@@ -6,5 +7,5 @@
             <plugin>gz_ros2_control/GazeboSimSystem</plugin>
         </hardware>
-        <!-- Declaração dos joints com interface de velocidade -->
+        <!-- Front Left Wheel Joint -->
         <joint name="front_left_wheel_joint">
             <command_interface name="velocity">
@@ -15,4 +16,5 @@
             <state_interface name="velocity"/>
         </joint>
+        <!-- Front Right Wheel Joint -->
         <joint name="front_right_wheel_joint">
             <command_interface name="velocity">
@@ -23,4 +25,5 @@
             <state_interface name="velocity"/>
         </joint>
+        <!-- Back Left Wheel Joint -->
         <joint name="back_left_wheel_joint">
             <command_interface name="velocity">
@@ -31,4 +34,5 @@
             <state_interface name="velocity"/>
         </joint>
+        <!-- Back Right Wheel Joint -->
         <joint name="back_right_wheel_joint">
             <command_interface name="velocity">
@@ -40,3 +44,13 @@
         </joint>
     </ros2_control>
+    <!-- Plugin para Gazebo Harmonic carregar os controladores -->
+    <gazebo>
+        <plugin filename="gz_ros2_control-system" name="gz_ros2_control::GazeboSimROS2ControlPlugin">
+            <parameters>$(find caramelo_controller)/config/robot_controllers.yaml</parameters>
+            <controller_manager_node_name>controller_manager</controller_manager_node_name>
+            <ros>
+                <remapping>/controller_manager/robot_description:=/robot_description</remapping>
+            </ros>
+        </plugin>
+    </gazebo>
 </robot>

Commit message: fixed robot URDF

File: src/caramelo_description/URDF/robot.urdf.xacro (robot description, xacro)
@@ -39,4 +39,4 @@
     y_reflect="-1"/>
   <!-- LiDAR (ajustado para as dimensões do YouBot) -->
-  <xacro:lidar_sensor parent="base_link" xyz="0.290 0.0 0.120" rpy="0 0 0"/>
+  <xacro:lidar_sensor parent="base_link" xyz="0.292 0.0 0.077" rpy="0 0 0"/>
 </robot>

File: src/caramelo_description/URDF/robot_base.xacro (robot description, xacro)
@@ -4,6 +4,8 @@
     <!-- Propriedades da base do robô Caramelo -->
     <xacro:property name="mass" value="22.0"/>
-    <xacro:property name="width" value="0.580"/>   <!-- Comprimento -->
-    <xacro:property name="depth" value="0.380"/>   <!-- Largura -->
+    <xacro:property name="width_vertical" value="0.550"/>   <!-- Comprimento -->
+    <xacro:property name="depth_vertical" value="0.210"/>   <!-- Largura -->
+    <xacro:property name="width_horizontal" value="0.330"/>   <!-- Comprimento -->
+    <xacro:property name="depth_horizontal" value="0.320"/>   <!-- Largura -->
     <xacro:property name="height" value="0.105"/>  <!-- Altura -->
     <xacro:property name="wheel_radius" value="0.05"/>
@@ -13,8 +15,17 @@
         <origin xyz="0 0 ${height/2.0}" rpy="0 0 0"/>
         <geometry>
-          <box size="${width} ${depth} ${height}"/>
+          <box size="${width_vertical} ${depth_vertical} ${height}"/>
         </geometry>
-        <material name="black">
-          <color rgba="0.0 0.0 0.0 1.0"/>
+        <material name="darkgray">
+          <color rgba="0.3 0.3 0.3 1.0"/>
+        </material>
+      </visual>
+      <visual>
+        <origin xyz="0 0 ${height/2.0}" rpy="0 0 0"/>
+        <geometry>
+          <box size="${depth_horizontal} ${width_horizontal} ${height}"/>
+        </geometry>
+        <material name="darkgray">
+          <color rgba="0.3 0.3 0.3 1.0"/>
         </material>
       </visual>
@@ -22,5 +33,5 @@
         <origin xyz="0 0 ${height/2.0}" rpy="0 0 0"/>
         <geometry>
-          <box size="${width} ${depth} ${height}"/>
+          <box size="${width_vertical} ${depth_vertical} ${height}"/>
         </geometry>
       </collision>
@@ -29,7 +40,7 @@
         <origin xyz="0 0 ${height/2.0}" rpy="0 0 0"/>
         <inertia
-          ixx="${1/12.0 * mass * (height*height + depth*depth)}"
-          iyy="${1/12.0 * mass * (width*width + depth*depth)}"
-          izz="${1/12.0 * mass * (width*width + height*height)}"
+          ixx="${1/12.0 * mass * (height*height + depth_vertical*depth_vertical)}"
+          iyy="${1/12.0 * mass * (width_vertical*width_vertical + depth_vertical*depth_vertical)}"
+          izz="${1/12.0 * mass * (width_vertical*width_vertical + height*height)}"
           ixy="0.0" ixz="0.0" iyz="0.0"/>
       </inertial>
@@ -45,6 +56,6 @@
       <visual>
         <material>
-          <ambient>0.0 0.0 0.0 1.0</ambient>
-          <diffuse>0.0 0.0 0.0 1.0</diffuse>
+          <ambient>0.3 0.3 0.3 1.0</ambient>
+          <diffuse>0.3 0.3 0.3 1.0</diffuse>
           <specular>0.1 0.1 0.1 1.0</specular>
           <emissive>0.0 0.0 0.0 1.0</emissive>

File: src/caramelo_description/URDF/robot_mecanum_wheel.xacro (robot description, xacro)
@@ -3,7 +3,7 @@
   <!-- Especificações das rodas mecanum do robô Caramelo -->
   <xacro:property name="wheel_radius" value="0.05" />
-  <xacro:property name="wheel_width" value="0.061" />
+  <xacro:property name="wheel_width" value="0.069" />
   <xacro:property name="wheel_mass" value="3.0" />
-  <xacro:property name="wheel_separation" value="0.370" />
+  <xacro:property name="wheel_separation" value="0.310" /> <!-- Distância entre as rodas 21 + 3 + 7 -->
   <xacro:property name="wheel_base" value="0.470" />
   <xacro:macro name="mecanum_wheel" params="prefix side x_reflect y_reflect">
@@ -11,10 +11,10 @@
       <!-- Geometria visual: roda como cilindro -->
       <visual>
-        <origin xyz="0 0 0" rpy="0 0 0"/>
+        <origin xyz="0 0 0" rpy="${pi/2} 0 0"/>
         <geometry>
           <cylinder radius="${wheel_radius}" length="${wheel_width}"/>
         </geometry>
-        <material name="wheel_material">
-          <color rgba="0.8 0.8 0.0 1.0"/>
+        <material name="orange">
+          <color rgba="1.0 0.5 0.0 1.0"/>
         </material>
       </visual>
@@ -41,13 +41,25 @@
       <parent link="${prefix}base_link"/>
       <child link="${prefix}${side}_wheel_link"/>
-      <origin xyz="${x_reflect*(wheel_base/2)} ${y_reflect*(wheel_separation/2)} 0" rpy="0 0 0"/>
+      <origin xyz="${x_reflect*(wheel_base/2)} ${y_reflect*(wheel_separation/2)} 0.02" rpy="0 0 0"/>
     </joint>
     <!-- Configurações específicas do Gazebo para as rodas mecanum -->
     <gazebo reference="${prefix}${side}_wheel_link">
-      <material>Gazebo/DarkGrey</material>
-      <!-- Propriedades de fricção básicas - configuração simplificada -->
-      <mu1>1.0</mu1>
-      <mu2>1.0</mu2>
-    </gazebo>
+      <surface>
+        <friction>
+          <ode>
+              <mu>1.0</mu>
+              <mu2>0.0</mu2>
+          </ode>
+        </friction>
+      </surface>
+      <visual>
+          <material>
+              <ambient>1.0 0.5 0.0 1.0</ambient>
+              <diffuse>1.0 0.5 0.0 1.0</diffuse>
+              <specular>0.2 0.2 0.2 1.0</specular>
+              <emissive>0.0 0.0 0.0 0.0</emissive>
+          </material>
+      </visual>
+  </gazebo>
   </xacro:macro>
 </robot>
