Commit message: teste com esferas

File: install/caramelo_simulation/share/caramelo_simulation/description/robot_core.xacro (robot description, xacro)
@@ -73,5 +73,7 @@
         <collision>
             <geometry>
-                <cylinder radius="0.05" length="0.075" />
+                <sphere>
+                    <radius>0.05</radius>
+                </sphere>
             </geometry>
         </collision>
@@ -101,5 +103,7 @@
         <collision>
             <geometry>
-                <cylinder radius="0.05" length="0.075" />
+                <sphere>
+                    <radius>0.05</radius>
+                </sphere>
             </geometry>
         </collision>
@@ -129,5 +133,7 @@
         <collision>
             <geometry>
-                <cylinder radius="0.05" length="0.075" />
+                <sphere>
+                    <radius>0.05</radius>
+                </sphere>
             </geometry>
         </collision>
@@ -157,5 +163,7 @@
         <collision>
             <geometry>
-                <cylinder radius="0.05" length="0.075" />
+                <sphere>
+                    <radius>0.05</radius>
+                </sphere>
             </geometry>
         </collision>

File: src/caramelo_description/URDF/robot_core.xacro (robot description, xacro)
@@ -80,4 +80,8 @@
     <gazebo reference="front_left_wheel">
         <material>Gazebo\Blue</material>
+        <mecanum_drive>
+            <roller_count>6</roller_count>
+            <roller_angle>45</roller_angle>
+        </mecanum_drive>
     </gazebo>
     <!--! FRONT RIGHT WHEEL -->
@@ -108,4 +112,8 @@
     <gazebo reference="front_right_wheel">
         <material>Gazebo\Blue</material>
+        <mecanum_drive>
+            <roller_count>6</roller_count>
+            <roller_angle>45</roller_angle>
+        </mecanum_drive>
     </gazebo>
     <!--! REAR LEFT WHEEL -->
@@ -136,4 +144,8 @@
     <gazebo reference="rear_left_wheel">
         <material>Gazebo\Blue</material>
+        <mecanum_drive>
+            <roller_count>6</roller_count>
+            <roller_angle>45</roller_angle>
+        </mecanum_drive>
     </gazebo>
     <!--! REAR RIGHT WHEEL -->
@@ -164,4 +176,8 @@
     <gazebo reference="rear_right_wheel">
         <material>Gazebo\Blue</material>
+        <mecanum_drive>
+            <roller_count>6</roller_count>
+            <roller_angle>45</roller_angle>
+        </mecanum_drive>
     </gazebo>
 </robot>

File: src/caramelo_description/URDF/robot_gazebo.xacro (robot description, xacro)
@@ -4,53 +4,85 @@
   <gazebo reference="fl_wheel_link">
     <collision>
-      <surface>
-        <friction>
-          <ode>
-            <mu>1.0</mu>
-            <mu2>0</mu2>
-            <fdir1 gz:expressed_in="base_footprint">1 -1 0</fdir1>
-          </ode>
-        </friction>
-      </surface>
+      <geometry>
+        <sphere>
+          <radius>0.05</radius> <!-- Define the radius of the sphere -->
+        </sphere>
+      </geometry>
     </collision>
+    <visual>
+      <geometry>
+        <cylinder>
+          <radius>0.05</radius>
+          <length>0.1</length>
+        </cylinder>
+      </geometry>
+    </visual>
+    <mecanum_drive>
+      <roller_count>6</roller_count>
+      <roller_angle>45</roller_angle>
+    </mecanum_drive>
   </gazebo>
   <gazebo reference="fr_wheel_link">
     <collision>
-      <surface>
-        <friction>
-          <ode>
-            <mu>1.0</mu>
-            <mu2>0</mu2>
-            <fdir1 gz:expressed_in="base_footprint">1 1 0</fdir1>
-          </ode>
-        </friction>
-      </surface>
+      <geometry>
+        <sphere>
+          <radius>0.05</radius>
+        </sphere>
+      </geometry>
     </collision>
+    <visual>
+      <geometry>
+        <cylinder>
+          <radius>0.05</radius>
+          <length>0.1</length>
+        </cylinder>
+      </geometry>
+    </visual>
+    <mecanum_drive>
+      <roller_count>6</roller_count>
+      <roller_angle>45</roller_angle>
+    </mecanum_drive>
   </gazebo>
   <gazebo reference="rl_wheel_link">
     <collision>
-      <surface>
-        <friction>
-          <ode>
-            <mu>0</mu>
-            <mu2>0</mu2>
-            <fdir1 gz:expressed_in="base_footprint">1 1 0</fdir1>
-          </ode>
-        </friction>
-      </surface>
+      <geometry>
+        <sphere>
+          <radius>0.05</radius>
+        </sphere>
+      </geometry>
     </collision>
+    <visual>
+      <geometry>
+        <cylinder>
+          <radius>0.05</radius>
+          <length>0.1</length>
+        </cylinder>
+      </geometry>
+    </visual>
+    <mecanum_drive>
+      <roller_count>6</roller_count>
+      <roller_angle>45</roller_angle>
+    </mecanum_drive>
   </gazebo>
   <gazebo reference="rr_wheel_link">
     <collision>
-      <surface>
-        <friction>
-          <ode>
-            <mu>0</mu>
-            <mu2>0</mu2>
-            <fdir1 gz:expressed_in="base_footprint">1 -1 0</fdir1>
-          </ode>
-        </friction>
-      </surface>
+      <geometry>
+        <sphere>
+          <radius>0.05</radius>
+        </sphere>
+      </geometry>
     </collision>
+    <visual>
+      <geometry>
+        <cylinder>
+          <radius>0.05</radius>
+          <length>0.1</length>
+        </cylinder>
+      </geometry>
+    </visual>
+    <mecanum_drive>
+      <roller_count>6</roller_count>
+      <roller_angle>45</roller_angle>
+    </mecanum_drive>
   </gazebo>
   <!-- Plugin ROS 2 Control Gazebo -->

File: src/caramelo_description/URDF/robot_ros2_control.xacro (robot description, xacro)
@@ -15,20 +15,24 @@
             </hardware>
         </xacro:unless>
-        <!-- Declaração dos joints com interface de velocidade -->
+        <!-- Definição dos joints com interfaces -->
         <joint name="fl_wheel_joint">
             <command_interface name="velocity" />
             <state_interface name="velocity" />
+            <state_interface name="position" />
         </joint>
         <joint name="fr_wheel_joint">
             <command_interface name="velocity" />
             <state_interface name="velocity" />
+            <state_interface name="position" />
         </joint>
         <joint name="rl_wheel_joint">
             <command_interface name="velocity" />
             <state_interface name="velocity" />
+            <state_interface name="position" />
         </joint>
         <joint name="rr_wheel_joint">
             <command_interface name="velocity" />
             <state_interface name="velocity" />
+            <state_interface name="position" />
         </joint>
     </ros2_control>
