Commit message: nav2 stack

File: src/caramelo_bringup/urdf/caramelo_real.urdf.xacro (robot description, xacro)
@@ -6,12 +6,13 @@
   <xacro:arg name="robot_name" default="caramelo"/>
   <xacro:arg name="prefix" default=""/>
-  <!-- Inclusões do caramelo_description (apenas visualização) -->
+  <!-- Argumento para Gazebo Ignition ou Gazebo Classic -->
+  <xacro:arg name="is_ignition" default="true"/>
+  <!-- Inclusões -->
   <xacro:include filename="$(find caramelo_description)/URDF/robot_base.xacro" />
   <xacro:include filename="$(find caramelo_description)/URDF/robot_mecanum_wheel.xacro" />
   <xacro:include filename="$(find caramelo_description)/URDF/lidar_sensor.xacro" />
-  <!-- base_footprint -->
-  <link name="base_footprint"/>
   <!-- Base -->
-  <xacro:robot_base parent="base_footprint"/>
+  <xacro:robot_base
+    prefix="$(arg prefix)"/>
   <!-- Rodas mecanum -->
   <xacro:mecanum_wheel
@@ -27,14 +28,22 @@
   <xacro:mecanum_wheel
     prefix="$(arg prefix)"
-    side="rear_left"
+    side="back_left"
     x_reflect="-1"
     y_reflect="1"/>
   <xacro:mecanum_wheel
     prefix="$(arg prefix)"
-    side="rear_right"
+    side="back_right"
     x_reflect="-1"
     y_reflect="-1"/>
-  <!-- LiDAR -->
-  <xacro:lidar_sensor parent="base_link" xyz="0.290 0.0 0.120" rpy="0 0 0"/>
+  <!-- RPLidar S2 - Posicionado na face frontal do robô -->
+  <xacro:lidar_sensor
+    prefix="$(arg prefix)"
+    parent="base_link"
+    frame_id="laser_frame"
+    xyz_offset="0.292 0 0.077"
+    rpy_offset="0 0 ${-M_PI}"
+    mesh_xyz_offset="0 0 0"
+    mesh_rpy_offset="0 0 0"
+    topic_name="scan"/>
   <!-- =============================================== -->
   <!-- ROS 2 Control Configuration for REAL HARDWARE -->

File: src/caramelo_description/URDF/lidar_sensor.xacro (robot description, xacro)
@@ -1,55 +1,108 @@
 <?xml version="1.0"?>
 <robot xmlns:xacro="http://www.ros.org/wiki/xacro">
-  <xacro:macro name="lidar_sensor" params="parent xyz rpy">
-    <link name="laser_frame">
+  <xacro:property name="M_PI" value="3.1415926535897931" />
+  <xacro:macro name="lidar_sensor" params="
+    prefix:=''
+    parent:='base_link'
+    frame_id:='laser_frame'
+    xyz_offset:='0 0 0'
+    rpy_offset:='0 0 0'
+    mesh_xyz_offset:='0 0 0'
+    mesh_rpy_offset:='${-M_PI/2} 0 0'
+    mesh_scale:='0.001 0.001 0.001'
+    collision_xyz_offset:='0 0 0'
+    collision_rpy_offset:='0 0 0'
+    inertial_xyz_offset:='0 0 0'
+    inertial_rpy_offset:='0 0 0'
+    lidar_width:=0.077
+    lidar_height:=0.0398
+    mass:=0.185
+    material_name:='rplidar_black'
+    material_color:='0.1 0.1 0.1 1'
+    gazebo_material_ambient:='0.1 0.1 0.1 1'
+    gazebo_material_diffuse:='0.1 0.1 0.1 1'
+    gazebo_material_specular:='0.1 0.1 0.1 1'
+    update_rate:=10
+    ray_count:=720
+    min_angle:='-3.14159'
+    max_angle:='3.14159'
+    min_range:='0.20'
+    max_range:='30.0'
+    range_resolution:='0.013'
+    topic_name:='scan'
+    always_on:=true
+    visualize:=false
+    enable_collision:=false">
+    <xacro:property name="radius" value="${lidar_width/2}" />
+    <xacro:property name="ixx_iyy" value="${(mass/12) * (3 * radius * radius + lidar_height * lidar_height)}" />
+    <xacro:property name="izz" value="${(mass/2) * (radius * radius)}" />
+    <link name="${prefix}${frame_id}">
       <visual>
+        <origin xyz="${mesh_xyz_offset}" rpy="${mesh_rpy_offset}"/>
         <geometry>
-          <cylinder length="0.016" radius="0.030" />
+          <cylinder radius="${lidar_width/2}" length="${lidar_height}"/>
         </geometry>
-        <origin xyz="0 0 0" rpy="0 0 0"/>
-        <material name="red" />
+        <material name="${material_name}">
+          <color rgba="${material_color}"/>
+        </material>
       </visual>
-      <collision>
-        <geometry>
-          <cylinder length="0.016" radius="0.030" />
-        </geometry>
-        <origin xyz="0 0 0" rpy="0 0 0"/>
-      </collision>
+      <xacro:if value="${enable_collision}">
+        <collision>
+          <origin xyz="${collision_xyz_offset}" rpy="${collision_rpy_offset}"/>
+          <geometry>
+            <cylinder radius="${lidar_width/2}" length="${lidar_height}"/>
+          </geometry>
+        </collision>
+      </xacro:if>
       <inertial>
-        <origin xyz="0 0 0" rpy="0 0 0"/>
-        <mass value="0.1"/>
+        <mass value="${mass}" />
+        <origin xyz="${inertial_xyz_offset}" rpy="${inertial_rpy_offset}"/>
         <inertia
-          ixx="1e-5" ixy="0.0" ixz="0.0"
-          iyy="1e-5" iyz="0.0"
-          izz="1e-5"/>
+          ixx="${ixx_iyy}"
+          ixy="0.0"
+          ixz="0.0"
+          iyy="${ixx_iyy}"
+          iyz="0.0"
+          izz="${izz}" />
       </inertial>
     </link>
-    <joint name="laser_joint" type="fixed">
-      <parent link="${parent}" />
-      <child link="laser_frame" />
-      <origin xyz="${xyz}" rpy="${rpy}" />
+    <joint name="${prefix}${frame_id}_joint" type="fixed">
+      <parent link="${prefix}${parent}"/>
+      <child link="${prefix}${frame_id}" />
+      <origin xyz="${xyz_offset}" rpy="${rpy_offset}"/>
     </joint>
-    <gazebo reference="laser_frame">
-      <sensor name="rplidar" type="ray">
-        <pose>0 0 0 0 0 0</pose>
-        <visualize>true</visualize>
-        <update_rate>10</update_rate>
+    <gazebo reference="${prefix}${frame_id}">
+      <material>
+        <ambient>${gazebo_material_ambient}</ambient>
+        <diffuse>${gazebo_material_diffuse}</diffuse>
+        <specular>${gazebo_material_specular}</specular>
+      </material>
+      <sensor name="${prefix}lidar_sensor" type="gpu_lidar">
+        <topic>${topic_name}</topic>
+        <update_rate>${update_rate}</update_rate>
+        <always_on>${always_on}</always_on>
+        <visualize>${visualize}</visualize>
         <ray>
           <scan>
             <horizontal>
-              <samples>360</samples>
-              <min_angle>-1.57</min_angle>
-              <max_angle>1.57</max_angle>
+              <samples>${ray_count}</samples>
+              <resolution>1</resolution>
+              <min_angle>${min_angle}</min_angle>
+              <max_angle>${max_angle}</max_angle>
             </horizontal>
+            <vertical>
+              <samples>1</samples>
+              <resolution>1</resolution>
+              <min_angle>0</min_angle>
+              <max_angle>0</max_angle>
+            </vertical>
           </scan>
           <range>
-            <min>0.3</min>
-            <max>20.0</max>
+            <min>${min_range}</min>
+            <max>${max_range}</max>
+            <resolution>${range_resolution}</resolution>
           </range>
         </ray>
-        <plugin name="gazebo_ros_ray_sensor" filename="libignition-gazebo-ros-ray-system.so">
-          <topic>/scan</topic>
-          <frame_name>laser_frame</frame_name>
-        </plugin>
+        <gz_frame_id>${prefix}${frame_id}</gz_frame_id>
       </sensor>
     </gazebo>

File: src/caramelo_description/URDF/robot.urdf.xacro (robot description, xacro)
@@ -13,8 +13,7 @@
   <xacro:include filename="$(find caramelo_description)/URDF/lidar_sensor.xacro" />
   <xacro:include filename="$(find caramelo_description)/URDF/robot_ros2_control.xacro" />
-  <!-- base_footprint -->
-  <link name="base_footprint"/>
   <!-- Base -->
-  <xacro:robot_base parent="base_footprint"/>
+  <xacro:robot_base
+    prefix="$(arg prefix)"/>
   <!-- Rodas mecanum -->
   <xacro:mecanum_wheel
@@ -38,5 +37,13 @@
     x_reflect="-1"
     y_reflect="-1"/>
-  <!-- LiDAR (ajustado para as dimensões do YouBot) -->
-  <xacro:lidar_sensor parent="base_link" xyz="0.292 0.0 0.077" rpy="0 0 0"/>
+  <!-- RPLidar S2 - Posicionado na face frontal do robô -->
+  <xacro:lidar_sensor
+    prefix="$(arg prefix)"
+    parent="base_link"
+    frame_id="laser_frame"
+    xyz_offset="0.292 0 0.077"
+    rpy_offset="0 0 ${-M_PI}"
+    mesh_xyz_offset="0 0 0"
+    mesh_rpy_offset="0 0 0"
+    topic_name="scan"/>
 </robot>

File: src/caramelo_description/URDF/robot_base.xacro (robot description, xacro)
@@ -1,15 +1,17 @@
 <?xml version="1.0"?>
 <robot xmlns:xacro="http://www.ros.org/wiki/xacro">
-  <xacro:macro name="robot_base" params="parent">
-    <!-- Propriedades da base do robô Caramelo -->
-    <xacro:property name="mass" value="22.0"/>
-    <xacro:property name="width_vertical" value="0.550"/>   <!-- Comprimento -->
-    <xacro:property name="depth_vertical" value="0.210"/>   <!-- Largura -->
-    <xacro:property name="width_horizontal" value="0.330"/>   <!-- Comprimento -->
-    <xacro:property name="depth_horizontal" value="0.320"/>   <!-- Largura -->
-    <xacro:property name="height" value="0.105"/>  <!-- Altura -->
-    <xacro:property name="wheel_radius" value="0.05"/>
+  <!-- Propriedades da base do robô Caramelo -->
+  <xacro:property name="mass" value="22.0"/>
+  <xacro:property name="width_vertical" value="0.550"/>   <!-- Comprimento -->
+  <xacro:property name="depth_vertical" value="0.210"/>   <!-- Largura -->
+  <xacro:property name="width_horizontal" value="0.330"/>   <!-- Comprimento -->
+  <xacro:property name="depth_horizontal" value="0.320"/>   <!-- Largura -->
+  <xacro:property name="height" value="0.105"/>  <!-- Altura -->
+  <xacro:property name="wheel_radius" value="0.05"/>
+  <xacro:macro name="robot_base" params="prefix">
+    <!-- BAsefootprint link -->
+    <link name="${prefix}base_footprint"/>
     <!-- Link da base (base_link agora toca o chão) -->
-    <link name="base_link">
+    <link name="${prefix}base_link">
       <visual>
         <origin xyz="0 0 ${height/2.0}" rpy="0 0 0"/>
@@ -47,11 +49,11 @@
     </link>
     <!-- Joint com o footprint (ajustado para as dimensões do Caramelo) -->
-    <joint name="base_joint" type="fixed">
-      <parent link="${parent}"/>
-      <child link="base_link"/>
-      <origin xyz="0 0 ${wheel_radius - 0.01}" rpy="0 0 0"/>
+    <joint name="${prefix}base_joint" type="fixed">
+      <parent link="${prefix}base_footprint"/>
+      <child link="${prefix}base_link"/>
+      <origin xyz="0 0 ${wheel_radius - 0.02}" rpy="0 0 0"/>
     </joint>
     <!-- Aparência no Gazebo -->
-    <gazebo reference="base_link">
+    <gazebo reference="${prefix}base_link">
       <visual>
         <material>

Commit message: fixed mappim odom topic and teleop

File: src/caramelo_bringup/urdf/caramelo_real.urdf.xacro (robot description, xacro)
@@ -75,5 +75,5 @@
     </joint>
     <!-- Joint para roda traseira esquerda -->
-    <joint name="rear_left_wheel_joint">
+    <joint name="back_left_wheel_joint">
       <command_interface name="velocity">
         <param name="min">-30.0</param>
@@ -84,5 +84,5 @@
     </joint>
     <!-- Joint para roda traseira direita -->
-    <joint name="rear_right_wheel_joint">
+    <joint name="back_right_wheel_joint">
       <command_interface name="velocity">
         <param name="min">-30.0</param>
